Commit message: update hand urdf

File: data/humanoid/hand.urdf (robot description, URDF)
Before this commit: robot dumpUrdf, 16 links, 15 joints
Links:
- link index_dist: mass 3.000000 -> 0.05
- link index_inter: mass 3.000000 -> 0.05
- link index_prox: mass 4.500000 -> 0.05
- link middle_dist: mass 3.000000 -> 0.05
- link middle_inter: mass 3.000000 -> 0.05
- link middle_prox: mass 4.500000 -> 0.05; geometry collision capsule length=0.120 radius=0.06
- link palm: mass 6.000000 -> 0.45; geometry collision box size=0.6 0.6 0.2
- link pinkie_dist: mass 3.000000 -> 0.05
- link pinkie_inter: mass 3.000000 -> 0.05
- link pinkie_prox: mass 4.500000 -> 0.05
- link ring_dist: mass 3.000000 -> 0.05
- link ring_inter: mass 3.000000 -> 0.05
- link ring_prox: mass 4.500000 -> 0.05
- link thumb_inter: mass 3.000000 -> 0.05
- link thumb_prox: mass 4.500000 -> 0.05
Joints:
- joint index_dist: axis 0.000000 0.000000 1.000000 -> 0.000000 1.000000 0.000000; limit lower=-3.14 upper=0. effort=1000.0 velocity=0.5 -> lower=0 upper=3.14 effort=1000.0 velocity=0.5; origin xyz=0.00000 0.00 0.000000 rpy=0 0 0 -> xyz=0.000000 -0.2400 0.000000 rpy=0 0 0
- joint index_inter: axis 0.000000 0.000000 1.000000 -> 0.000000 1.000000 0.000000; origin xyz=0.00000 0.00 0.000000 rpy=0 0 0 -> xyz=0.000000 -0.2400 0.000000 rpy=0 0 0
- joint index_prox: origin xyz=0.0800000 -0.36000 0.0 rpy=0 0 0 -> xyz=0.2000 -0.66000 0.0 rpy=0 0 0
- joint middle_dist: axis 0.000000 0.000000 1.000000 -> 0.000000 1.000000 0.000000; limit lower=-3.14 upper=0. effort=1000.0 velocity=0.5 -> lower=0 upper=3.14 effort=1000.0 velocity=0.5; origin xyz=0.000000 0.00 0.000000 rpy=0 0 0 -> xyz=0.000000 -0.2400 0.000000 rpy=0 0 0
- joint middle_inter: axis 0.000000 0.000000 1.000000 -> 0.000000 1.000000 0.000000; limit lower=-3.14 upper=0. effort=1000.0 velocity=0.5 -> lower=0 upper=3.14 effort=1000.0 velocity=0.5; origin xyz=0.000000 0.00 0.000000 rpy=0 0 0 -> xyz=0.000000 -0.2400 0.000000 rpy=0 0 0
- joint middle_prox: origin xyz=0.00000 -0.36000 0.0 rpy=0 0 0 -> xyz=0.08000 -0.66000 0.0 rpy=0 0 0
- joint palm: origin xyz=0.000000 0.000000 0.000000 rpy=-1.57 0 0 -> xyz=0.000000 0.000000 0.000000 rpy=0 0 0
- joint pinkie_dist: axis 0.000000 0.000000 1.000000 -> 0.000000 1.000000 0.000000; limit lower=-3.14 upper=0. effort=1000.0 velocity=0.5 -> lower=0 upper=3.14 effort=1000.0 velocity=0.5; origin xyz=0.000000 0.00 0.000000 rpy=0 0 0 -> xyz=0.000000 -0.2400 0.000000 rpy=0 0 0
- joint pinkie_inter: axis 0.000000 0.000000 1.000000 -> 0.000000 1.000000 0.000000; limit lower=-3.14 upper=0. effort=1000.0 velocity=0.5 -> lower=0 upper=3.14 effort=1000.0 velocity=0.5; origin xyz=0.000000 0.00 0.000000 rpy=0 0 0 -> xyz=0.000000 -0.2400 0.000000 rpy=0 0 0
- joint pinkie_prox: origin xyz=-0.160000 -0.36000 0.0 rpy=0 0 0 -> xyz=-0.1600 -0.66000 0.0 rpy=0 0 0
- joint ring_dist: axis 0.000000 0.000000 1.000000 -> 0.000000 1.000000 0.000000; limit lower=-3.14 upper=0. effort=1000.0 velocity=0.5 -> lower=0 upper=3.14 effort=1000.0 velocity=0.5; origin xyz=0.000000 0.00 0.000000 rpy=0 0 0 -> xyz=0.000000 -0.2400 0.000000 rpy=0 0 0
- joint ring_inter: axis 0.000000 0.000000 1.000000 -> 0.000000 1.000000 0.000000; limit lower=-3.14 upper=0. effort=1000.0 velocity=0.5 -> lower=0 upper=3.14 effort=1000.0 velocity=0.5; origin xyz=0.000000 0.00 0.000000 rpy=0 0 0 -> xyz=0.000000 -0.2400 0.000000 rpy=0 0 0
- joint ring_prox: origin xyz=-0.080000 -0.36000 0.0 rpy=0 0 0 -> xyz=-0.04000 -0.66000 0.0 rpy=0 0 0
- joint thumb_inter: axis 0.000000 0.000000 1.000000 -> 0.000000 1.000000 0.000000; limit lower=-3.14 upper=0. effort=1000.0 velocity=0.5 -> lower=0 upper=3.14 effort=1000.0 velocity=0.5; origin xyz=0.000000 0.00 0.000000 rpy=0 0 0 -> xyz=0.2400 0.00 0.000000 rpy=0 0 0
- joint thumb_prox: origin xyz=0.00000 -0.42000 0.0 rpy=0 1.57 1.57 -> xyz=0.3000 -0.360 0.0 rpy=0 0 0
