Commit message: update

File: data/humanoid/new_simple_hand.urdf (robot description, URDF)
Before this commit: robot dumpUrdf, 16 links, 15 joints
Links:
- removed link palm
- added link thumb_dist, mass 0.05; collision box size=0.05 0.05 0.1
- added link wrist, mass 0.1; collision box size=0.05 0.05 0.05
- link index_dist: geometry collision box size=0.05 0.05 0.1
- link index_inter: geometry collision box size=0.05 0.05 0.1
- link index_prox: geometry collision box size=0.05 0.05 0.1
- link middle_dist: geometry collision box size=0.05 0.05 0.1
- link middle_inter: geometry collision box size=0.05 0.05 0.1
- link middle_prox: geometry collision box size=0.05 0.05 0.1
- link pinkie_dist: geometry collision box size=0.05 0.05 0.1
- link pinkie_inter: geometry collision box size=0.05 0.05 0.1
- link pinkie_prox: geometry collision box size=0.05 0.05 0.1
- link ring_dist: geometry collision box size=0.05 0.05 0.1
- link ring_inter: geometry collision box size=0.05 0.05 0.1
- link ring_prox: geometry collision box size=0.05 0.05 0.1
- link thumb_inter: geometry collision box size=0.05 0.05 0.1
- link thumb_prox: geometry collision box size=0.05 0.05 0.1
Joints:
- removed joint palm
- added joint thumb_dist: type revolute, parent thumb_inter, child thumb_dist, origin xyz=0.10562241077423096 -0.005341768264770508 0.13189956545829773 rpy=0 0 0, axis 0.000000 1.000000 0.000000, limit lower=-3.14 upper=3.14 effort=1000.0 velocity=0.5
- added joint wrist: type fixed, parent base, child wrist, origin xyz=0 0 0 rpy=3.14 -1.57 1.57
- joint index_dist: origin xyz=0.000000 -0.2400 0.000000 rpy=0 0 0 -> xyz=-0.0008243322372436523 0.028004944324493408 0.12339383363723755 rpy=0 0 0
- joint index_inter: origin xyz=0.000000 -0.2400 0.000000 rpy=0 0 0 -> xyz=-0.0012820959091186523 0.030645132064819336 0.12021106481552124 rpy=0 0 0
- joint index_prox: axis (none) -> 1.000000 0.000000 0.000000; limit (none) -> lower=-3.14 upper=3.14 effort=1000 velocity=0.5; origin xyz=0.2000 -0.66000 0.0 rpy=0 0 0 -> xyz=0.0691772997379303 0.16612380743026733 0.6951615214347839 rpy=0 0 0; parent palm -> wrist; type spherical -> revolute
- joint middle_dist: origin xyz=0.000000 -0.2400 0.000000 rpy=0 0 0 -> xyz=-0.020906776189804077 0.024646222591400146 0.12368118762969971 rpy=0 0 0
- joint middle_inter: origin xyz=0.000000 -0.2400 0.000000 rpy=0 0 0 -> xyz=-0.024123787879943848 0.04249602556228638 0.12114346027374268 rpy=0 0 0
- joint middle_prox: axis (none) -> 1.000000 0.000000 0.000000; limit (none) -> lower=-3.14 upper=3.14 effort=1000 velocity=0.5; origin xyz=0.08000 -0.66000 0.0 rpy=0 0 0 -> xyz=-0.08907824754714966 0.19644707441329956 0.7083621025085449 rpy=0 0 0; parent palm -> wrist; type spherical -> revolute
- joint pinkie_dist: origin xyz=0.000000 -0.2400 0.000000 rpy=0 0 0 -> xyz=-0.040886253118515015 0.006254315376281738 0.08677315711975098 rpy=0 0 0
- joint pinkie_inter: origin xyz=0.000000 -0.2400 0.000000 rpy=0 0 0 -> xyz=-0.05650430917739868 0.011394917964935303 0.08920609951019287 rpy=0 0 0
- joint pinkie_prox: axis (none) -> 1.000000 0.000000 0.000000; limit (none) -> lower=-3.14 upper=3.14 effort=1000 velocity=0.5; origin xyz=-0.1600 -0.66000 0.0 rpy=0 0 0 -> xyz=-0.30925989151000977 0.1727619767189026 0.501175045967102 rpy=0 0 0; parent palm -> wrist; type spherical -> revolute
- joint ring_dist: origin xyz=0.000000 -0.2400 0.000000 rpy=0 0 0 -> xyz=-0.03399193286895752 7.867813110351562e-05 0.10368543863296509 rpy=0 0 0
- joint ring_inter: origin xyz=0.000000 -0.2400 0.000000 rpy=0 0 0 -> xyz=-0.04373997449874878 0.03548264503479004 0.11856430768966675 rpy=0 0 0
- joint ring_prox: axis (none) -> 1.000000 0.000000 0.000000; limit (none) -> lower=-3.14 upper=3.14 effort=1000 velocity=0.5; origin xyz=-0.04000 -0.66000 0.0 rpy=0 0 0 -> xyz=-0.20733147859573364 0.18892675638198853 0.6320534348487854 rpy=0 0 0; parent palm -> wrist; type spherical -> revolute
- joint thumb_inter: origin xyz=0.2400 0.00 0.000000 rpy=0 0 0 -> xyz=0.08786723017692566 0.01713097095489502 0.11243215203285217 rpy=0 0 0
- joint thumb_prox: axis (none) -> 0.000000 1.000000 0.000000; limit (none) -> lower=-3.14 upper=3.14 effort=1000 velocity=0.5; origin xyz=0.3000 -0.360 0.0 rpy=0 0 0 -> xyz=0.25435328483581543 0.16699939966201782 0.31131690740585327 rpy=1.57 0 0; parent palm -> wrist; type spherical -> revolute

Commit message: update with working controller

File: data/humanoid/new_simple_hand.urdf (robot description, URDF)
Before this commit: robot dumpUrdf, 17 links, 16 joints
Joints:
- joint index_dist: limit lower=-3.14 upper=3.14 effort=1000.0 velocity=0.5 -> lower=0 upper=1.57 effort=1000.0 velocity=0.5
- joint index_inter: limit lower=-3.14 upper=3.14 effort=1000.0 velocity=0.5 -> lower=0 upper=1.57 effort=1000.0 velocity=0.5
- joint index_prox: limit lower=-3.14 upper=3.14 effort=1000 velocity=0.5 -> lower=0 upper=1.57 effort=1000 velocity=0.5
- joint middle_dist: limit lower=-3.14 upper=3.14 effort=1000.0 velocity=0.5 -> lower=0 upper=1.57 effort=1000.0 velocity=0.5
- joint middle_inter: limit lower=-3.14 upper=3.14 effort=1000.0 velocity=0.5 -> lower=0 upper=1.57 effort=1000.0 velocity=0.5
- joint middle_prox: limit lower=-3.14 upper=3.14 effort=1000 velocity=0.5 -> lower=0 upper=1.57 effort=1000 velocity=0.5
- joint pinkie_dist: limit lower=-3.14 upper=3.14 effort=1000.0 velocity=0.5 -> lower=0 upper=1.57 effort=1000.0 velocity=0.5
- joint pinkie_inter: limit lower=-3.14 upper=3.14 effort=1000.0 velocity=0.5 -> lower=0 upper=1.57 effort=1000.0 velocity=0.5
- joint pinkie_prox: limit lower=-3.14 upper=3.14 effort=1000 velocity=0.5 -> lower=0 upper=1.57 effort=1000 velocity=0.5
- joint ring_dist: limit lower=-3.14 upper=3.14 effort=1000.0 velocity=0.5 -> lower=0 upper=1.57 effort=1000.0 velocity=0.5
- joint ring_inter: limit lower=-3.14 upper=3.14 effort=1000.0 velocity=0.5 -> lower=0 upper=1.57 effort=1000.0 velocity=0.5
- joint ring_prox: limit lower=-3.14 upper=3.14 effort=1000 velocity=0.5 -> lower=0 upper=1.57 effort=1000 velocity=0.5
- joint thumb_dist: limit lower=-3.14 upper=3.14 effort=1000.0 velocity=0.5 -> lower=0 upper=1.57 effort=1000.0 velocity=0.5
- joint thumb_inter: limit lower=-3.14 upper=3.14 effort=1000.0 velocity=0.5 -> lower=0 upper=1.57 effort=1000.0 velocity=0.5
- joint thumb_prox: limit lower=-3.14 upper=3.14 effort=1000 velocity=0.5 -> lower=0 upper=1.57 effort=1000 velocity=0.5; origin xyz=0.25435328483581543 0.16699939966201782 0.31131690740585327 rpy=1.57 0 0 -> xyz=0.25435328483581543 0.16699939966201782 0.31131690740585327 rpy=0 0 0
