Commit message: update hand model

File: data/humanoid/old_new_simple_hand.urdf (robot description, URDF)
Before this commit: robot dumpUrdf, 17 links, 16 joints
Links:
- link index_dist: geometry collision box size=0.05 0.05 0.1
- link index_inter: geometry collision box size=0.05 0.05 0.1
- link index_prox: geometry collision box size=0.05 0.05 0.1
- link middle_dist: geometry collision box size=0.05 0.05 0.1
- link middle_inter: geometry collision box size=0.05 0.05 0.1
- link middle_prox: geometry collision box size=0.05 0.05 0.1
- link pinkie_dist: geometry collision box size=0.05 0.05 0.1
- link pinkie_inter: geometry collision box size=0.05 0.05 0.1
- link pinkie_prox: geometry collision box size=0.05 0.05 0.1
- link ring_dist: geometry collision box size=0.05 0.05 0.1
- link ring_inter: geometry collision box size=0.05 0.05 0.1
- link ring_prox: geometry collision box size=0.05 0.05 0.1
- link thumb_dist: geometry collision box size=0.05 0.05 0.1
- link thumb_inter: geometry collision box size=0.05 0.05 0.1
- link thumb_prox: geometry collision box size=0.05 0.05 0.1
Joints:
- joint index_dist: origin xyz=0 0 0.12339383363723755 rpy=0 0 0 -> xyz=-0.0008243322372436523 0.028004944324493408 0.12339383363723755 rpy=0 0 0
- joint index_inter: origin xyz=0 0 0.12021106481552124 rpy=0 0 0 -> xyz=-0.0012820959091186523 0.030645132064819336 0.12021106481552124 rpy=0 0 0
- joint middle_dist: origin xyz=0 0 0.12368118762969971 rpy=0 0 0 -> xyz=-0.020906776189804077 0.024646222591400146 0.12368118762969971 rpy=0 0 0
- joint middle_inter: origin xyz=0 0 0.12114346027374268 rpy=0 0 0 -> xyz=-0.024123787879943848 0.04249602556228638 0.12114346027374268 rpy=0 0 0
- joint middle_prox: origin xyz=-0.08907824754714966 0.19644707441329956 0.7083621025085449 rpy=0 0 0.1 -> xyz=-0.08907824754714966 0.19644707441329956 0.7083621025085449 rpy=0 0 0
- joint pinkie_dist: origin xyz=0 0 0.08677315711975098 rpy=0 0 0 -> xyz=-0.040886253118515015 0.006254315376281738 0.08677315711975098 rpy=0 0 0
- joint pinkie_inter: origin xyz=0 0 0.08920609951019287 rpy=0 0 0 -> xyz=-0.05650430917739868 0.011394917964935303 0.08920609951019287 rpy=0 0 0
- joint pinkie_prox: origin xyz=-0.30925989151000977 0.1727619767189026 0.501175045967102 rpy=0 -0.13 0.21 -> xyz=-0.30925989151000977 0.1727619767189026 0.501175045967102 rpy=0 0 0
- joint ring_dist: origin xyz=0 0 0.10368543863296509 rpy=0 0 0 -> xyz=-0.03399193286895752 7.867813110351562e-05 0.10368543863296509 rpy=0 0 0
- joint ring_inter: origin xyz=0 0 0.11856430768966675 rpy=0 0 0 -> xyz=-0.04373997449874878 0.03548264503479004 0.11856430768966675 rpy=0 0 0
- joint ring_prox: origin xyz=-0.20733147859573364 0.18892675638198853 0.6320534348487854 rpy=0 -0.05 0.11 -> xyz=-0.20733147859573364 0.18892675638198853 0.6320534348487854 rpy=0 0 0
- joint thumb_dist: origin xyz=0 0 0.13189956545829773 rpy=0 0 0 -> xyz=0.10562241077423096 -0.005341768264770508 0.13189956545829773 rpy=0 0 0
- joint thumb_inter: origin xyz=0 0 0.11243215203285217 rpy=0 0 0 -> xyz=0.08786723017692566 0.01713097095489502 0.11243215203285217 rpy=0 0 0
- joint thumb_prox: origin xyz=0.25435328483581543 0.16699939966201782 0.31131690740585327 rpy=3.14 -1.47 0 -> xyz=0.25435328483581543 0.16699939966201782 0.31131690740585327 rpy=0 0 0
