Commit message: add whole humanoid

File: data/humanoid/whole_upper_humanoid.urdf (robot description, URDF)
Before this commit: robot dumpUrdf, 31 links, 30 joints
Links:
- removed link index_dist
- removed link index_inter
- removed link index_prox
- removed link middle_dist
- removed link middle_inter
- removed link middle_prox
- removed link pinkie_dist
- removed link pinkie_inter
- removed link pinkie_prox
- removed link ring_dist
- removed link ring_inter
- removed link ring_prox
- removed link thumb_dist
- removed link thumb_inter
- removed link thumb_prox
- added link l_index_dist, mass 0.05; collision box size=0.025 0.025 0.04
- added link l_index_inter, mass 0.05; collision box size=0.025 0.025 0.04
- added link l_index_prox, mass 0.05; collision box size=0.025 0.025 0.04
- added link l_middle_dist, mass 0.05; collision box size=0.025 0.025 0.04
- added link l_middle_inter, mass 0.05; collision box size=0.025 0.025 0.04
- added link l_middle_prox, mass 0.05; collision box size=0.025 0.025 0.04
- added link l_pinkie_dist, mass 0.05; collision box size=0.025 0.025 0.04
- added link l_pinkie_inter, mass 0.05; collision box size=0.025 0.025 0.04
- added link l_pinkie_prox, mass 0.05; collision box size=0.025 0.025 0.04
- added link l_ring_dist, mass 0.05; collision box size=0.025 0.025 0.04
- added link l_ring_inter, mass 0.05; collision box size=0.025 0.025 0.04
- added link l_ring_prox, mass 0.05; collision box size=0.025 0.025 0.04
- added link l_thumb_dist, mass 0.05; collision box size=0.025 0.025 0.04
- added link l_thumb_inter, mass 0.05; collision box size=0.025 0.025 0.04
- added link l_thumb_prox, mass 0.05; collision box size=0.025 0.025 0.04
- added link r_index_dist, mass 0.05; collision box size=0.025 0.025 0.04
- added link r_index_inter, mass 0.05; collision box size=0.025 0.025 0.04
- added link r_index_prox, mass 0.05; collision box size=0.025 0.025 0.04
- added link r_middle_dist, mass 0.05; collision box size=0.025 0.025 0.04
- added link r_middle_inter, mass 0.05; collision box size=0.025 0.025 0.04
- added link r_middle_prox, mass 0.05; collision box size=0.025 0.025 0.04
- added link r_pinkie_dist, mass 0.05; collision box size=0.025 0.025 0.04
- added link r_pinkie_inter, mass 0.05; collision box size=0.025 0.025 0.04
- added link r_pinkie_prox, mass 0.05; collision box size=0.025 0.025 0.04
- added link r_ring_dist, mass 0.05; collision box size=0.025 0.025 0.04
- added link r_ring_inter, mass 0.05; collision box size=0.025 0.025 0.04
- added link r_ring_prox, mass 0.05; collision box size=0.025 0.025 0.04
- added link r_thumb_dist, mass 0.05; collision box size=0.025 0.025 0.04
- added link r_thumb_inter, mass 0.05; collision box size=0.025 0.025 0.04
- added link r_thumb_prox, mass 0.05; collision box size=0.025 0.025 0.04
- link left_wrist: geometry collision box size=0.15 0.04 0.15
- link right_wrist: geometry collision box size=0.15 0.04 0.15
Joints:
- removed joint index_dist
- removed joint index_inter
- removed joint index_prox
- removed joint middle_dist
- removed joint middle_inter
- removed joint middle_prox
- removed joint pinkie_dist
- removed joint pinkie_inter
- removed joint pinkie_prox
- removed joint ring_dist
- removed joint ring_inter
- removed joint ring_prox
- removed joint thumb_dist
- removed joint thumb_inter
- removed joint thumb_prox
- added joint l_index_dist: type revolute, parent l_index_inter, child l_index_dist, origin xyz=0 0 0.061 rpy=0 0 0, axis 1.000000 0.000000 0.000000, limit lower=0 upper=2 effort=1000.0 velocity=0.5
- added joint l_index_inter: type revolute, parent l_index_prox, child l_index_inter, origin xyz=0 0 0.061 rpy=0 0 0, axis 1.000000 0.000000 0.000000, limit lower=0 upper=2 effort=1000.0 velocity=0.5
- added joint l_index_prox: type revolute, parent left_wrist, child l_index_prox, origin xyz=0.08 0 0.22 rpy=0 0 0, axis 1.000000 0.000000 0.000000, limit lower=0 upper=2 effort=1000 velocity=0.5
- added joint l_middle_dist: type revolute, parent l_middle_inter, child l_middle_dist, origin xyz=0 0 0.062 rpy=0 0 0, axis 1.000000 0.000000 0.000000, limit lower=0 upper=2 effort=1000.0 velocity=0.5
- added joint l_middle_inter: type revolute, parent l_middle_prox, child l_middle_inter, origin xyz=0 0 0.060 rpy=0 0 0, axis 1.000000 0.000000 0.000000, limit lower=0 upper=2 effort=1000.0 velocity=0.5
- added joint l_middle_prox: type revolute, parent left_wrist, child l_middle_prox, origin xyz=0.01 0 0.227 rpy=0 0 0.1, axis 1.000000 0.000000 0.000000, limit lower=0 upper=2 effort=1000 velocity=0.5
- added joint l_pinkie_dist: type revolute, parent l_pinkie_inter, child l_pinkie_dist, origin xyz=0 0 0.044 rpy=0 0 0, axis 1.000000 0.000000 0.000000, limit lower=0 upper=2 effort=1000.0 velocity=0.5
- added joint l_pinkie_inter: type revolute, parent l_pinkie_prox, child l_pinkie_inter, origin xyz=0 0 0.045 rpy=0 0 0, axis 1.000000 0.000000 0.000000, limit lower=0 upper=2 effort=1000.0 velocity=0.5
- added joint l_pinkie_prox: type revolute, parent left_wrist, child l_pinkie_prox, origin xyz=-0.108 0 0.123 rpy=0 -0.13 0.21, axis 1.000000 0.000000 0.000000, limit lower=0 upper=2 effort=1000 velocity=0.5
- added joint l_ring_dist: type revolute, parent l_ring_inter, child l_ring_dist, origin xyz=0 0 0.052 rpy=0 0 0, axis 1.000000 0.000000 0.000000, limit lower=0 upper=2 effort=1000.0 velocity=0.5
- added joint l_ring_inter: type revolute, parent l_ring_prox, child l_ring_inter, origin xyz=0 0 0.059 rpy=0 0 0, axis 1.000000 0.000000 0.000000, limit lower=0 upper=2 effort=1000.0 velocity=0.5
- added joint l_ring_prox: type revolute, parent left_wrist, child l_ring_prox, origin xyz=-0.057 0 0.189 rpy=0 -0.05 0.11, axis 1.000000 0.000000 0.000000, limit lower=0 upper=2 effort=1000 velocity=0.5
- added joint l_thumb_dist: type revolute, parent l_thumb_inter, child l_thumb_dist, origin xyz=0 0 0.066 rpy=0 0 0, axis 0.000000 1.000000 0.000000, limit lower=0 upper=2 effort=1000.0 velocity=0.5
- added joint l_thumb_inter: type revolute, parent l_thumb_prox, child l_thumb_inter, origin xyz=0 0 0.056 rpy=0 0 0, axis 0.000000 1.000000 0.000000, limit lower=0 upper=2 effort=1000.0 velocity=0.5
- added joint l_thumb_prox: type revolute, parent left_wrist, child l_thumb_prox, origin xyz=0.1 0 0 rpy=3.14 -2.81 0, axis 0.000000 1.000000 0.000000, limit lower=0 upper=2 effort=1000 velocity=0.5
- added joint r_index_dist: type revolute, parent r_index_inter, child r_index_dist, origin xyz=0 0 0.061 rpy=0 0 0, axis 1.000000 0.000000 0.000000, limit lower=0 upper=2 effort=1000.0 velocity=0.5
- added joint r_index_inter: type revolute, parent r_index_prox, child r_index_inter, origin xyz=0 0 0.061 rpy=0 0 0, axis 1.000000 0.000000 0.000000, limit lower=0 upper=2 effort=1000.0 velocity=0.5
- added joint r_index_prox: type revolute, parent right_wrist, child r_index_prox, origin xyz=0.08 0 0.22 rpy=0 0 0, axis 1.000000 0.000000 0.000000, limit lower=0 upper=2 effort=1000 velocity=0.5
- added joint r_middle_dist: type revolute, parent r_middle_inter, child r_middle_dist, origin xyz=0 0 0.062 rpy=0 0 0, axis 1.000000 0.000000 0.000000, limit lower=0 upper=2 effort=1000.0 velocity=0.5
- added joint r_middle_inter: type revolute, parent r_middle_prox, child r_middle_inter, origin xyz=0 0 0.060 rpy=0 0 0, axis 1.000000 0.000000 0.000000, limit lower=0 upper=2 effort=1000.0 velocity=0.5
- added joint r_middle_prox: type revolute, parent right_wrist, child r_middle_prox, origin xyz=0.01 0 0.227 rpy=0 0 0.1, axis 1.000000 0.000000 0.000000, limit lower=0 upper=2 effort=1000 velocity=0.5
- added joint r_pinkie_dist: type revolute, parent r_pinkie_inter, child r_pinkie_dist, origin xyz=0 0 0.044 rpy=0 0 0, axis 1.000000 0.000000 0.000000, limit lower=0 upper=2 effort=1000.0 velocity=0.5
- added joint r_pinkie_inter: type revolute, parent r_pinkie_prox, child r_pinkie_inter, origin xyz=0 0 0.045 rpy=0 0 0, axis 1.000000 0.000000 0.000000, limit lower=0 upper=2 effort=1000.0 velocity=0.5
- added joint r_pinkie_prox: type revolute, parent right_wrist, child r_pinkie_prox, origin xyz=-0.108 0 0.123 rpy=0 -0.13 0.21, axis 1.000000 0.000000 0.000000, limit lower=0 upper=2 effort=1000 velocity=0.5
- added joint r_ring_dist: type revolute, parent r_ring_inter, child r_ring_dist, origin xyz=0 0 0.052 rpy=0 0 0, axis 1.000000 0.000000 0.000000, limit lower=0 upper=2 effort=1000.0 velocity=0.5
- added joint r_ring_inter: type revolute, parent r_ring_prox, child r_ring_inter, origin xyz=0 0 0.059 rpy=0 0 0, axis 1.000000 0.000000 0.000000, limit lower=0 upper=2 effort=1000.0 velocity=0.5
- added joint r_ring_prox: type revolute, parent right_wrist, child r_ring_prox, origin xyz=-0.057 0 0.189 rpy=0 -0.05 0.11, axis 1.000000 0.000000 0.000000, limit lower=0 upper=2 effort=1000 velocity=0.5
- added joint r_thumb_dist: type revolute, parent r_thumb_inter, child r_thumb_dist, origin xyz=0 0 0.066 rpy=0 0 0, axis 0.000000 1.000000 0.000000, limit lower=0 upper=2 effort=1000.0 velocity=0.5
- added joint r_thumb_inter: type revolute, parent r_thumb_prox, child r_thumb_inter, origin xyz=0 0 0.056 rpy=0 0 0, axis 0.000000 1.000000 0.000000, limit lower=0 upper=2 effort=1000.0 velocity=0.5
- added joint r_thumb_prox: type revolute, parent right_wrist, child r_thumb_prox, origin xyz=0.1 0 0 rpy=3.14 -2.81 0, axis 0.000000 1.000000 0.000000, limit lower=0 upper=2 effort=1000 velocity=0.5
- joint left_wrist: axis (none) -> 1.000000 0.000000 0.000000; limit (none) -> lower=-1.57 upper=1.57 effort=1000.0 velocity=0.5; origin xyz=0.000000 -1.035788 0.000000 rpy=0 0 0 -> xyz=0.000000 -1.035788 0.000000 rpy=1.57 0 0; type fixed -> revolute
- joint right_wrist: axis (none) -> 1.000000 0.000000 0.000000; limit (none) -> lower=-1.57 upper=1.57 effort=1000.0 velocity=0.5; type spherical -> revolute

Commit message: update to working baseline

File: data/humanoid/whole_upper_humanoid.urdf (robot description, URDF)
Before this commit: robot dumpUrdf, 46 links, 45 joints
Joints:
- joint l_index_dist: axis 1.000000 0.000000 0.000000 -> -1.000000 0.000000 0.000000
- joint l_index_inter: axis 1.000000 0.000000 0.000000 -> -1.000000 0.000000 0.000000
- joint l_index_prox: axis 1.000000 0.000000 0.000000 -> -1.000000 0.000000 0.000000
- joint l_middle_dist: axis 1.000000 0.000000 0.000000 -> -1.000000 0.000000 0.000000
- joint l_middle_inter: axis 1.000000 0.000000 0.000000 -> -1.000000 0.000000 0.000000
- joint l_middle_prox: axis 1.000000 0.000000 0.000000 -> -1.000000 0.000000 0.000000
- joint l_pinkie_dist: axis 1.000000 0.000000 0.000000 -> -1.000000 0.000000 0.000000
- joint l_pinkie_inter: axis 1.000000 0.000000 0.000000 -> -1.000000 0.000000 0.000000
- joint l_pinkie_prox: axis 1.000000 0.000000 0.000000 -> -1.000000 0.000000 0.000000
- joint l_ring_dist: axis 1.000000 0.000000 0.000000 -> -1.000000 0.000000 0.000000
- joint l_ring_inter: axis 1.000000 0.000000 0.000000 -> -1.000000 0.000000 0.000000
- joint l_ring_prox: axis 1.000000 0.000000 0.000000 -> -1.000000 0.000000 0.000000
- joint left_shoulder: origin xyz=-0.096200 0.974000 -0.732440 rpy=0 0 0 -> xyz=-0.096200 0.974000 -0.732440 rpy=1.57 0 0
- joint right_shoulder: origin xyz=-0.096200 0.974000 0.732440 rpy=0 0 0 -> xyz=-0.096200 0.974000 0.732440 rpy=-1.57 0 0

Commit message: update start position of shoulders

File: data/humanoid/whole_upper_humanoid.urdf (robot description, URDF)
Before this commit: robot dumpUrdf, 46 links, 45 joints
Joints:
- joint left_shoulder: origin xyz=-0.096200 0.974000 -0.732440 rpy=1.57 0 0 -> xyz=-0.096200 0.974000 -0.732440 rpy=0 0 0
- joint right_shoulder: origin xyz=-0.096200 0.974000 0.732440 rpy=-1.57 0 0 -> xyz=-0.096200 0.974000 0.732440 rpy=0 0 0

Commit message: update weights of ankles to stabilise character

File: data/humanoid/whole_upper_humanoid.urdf (robot description, URDF)
Before this commit: robot dumpUrdf, 46 links, 45 joints
Links:
- link left_ankle: mass 100.000000 -> 1000
- link left_hip: mass 4.500000 -> 4.5
- link left_knee: mass 3.000000 -> 3.0
- link right_ankle: mass 100.000000 -> 1000
- link right_hip: mass 4.500000 -> 4.5
- link right_knee: mass 3.000000 -> 3.0
